File: _autosave-safetbutton.sch (KiCad schematic (older format))
At the start: 26 parts, among them J1 Conn_01x02_Male, J3 Conn_01x02_Male, J4 Conn_01x02_Male, J5 Conn_01x01_Male, J6 Conn_01x01_Male, J7 Conn_ARM_JTAG_SWD_10, Q1 Q_PMOS_GDSD, Q2 BSS138, U1 LP2985-2.8, U3 BC805M

Commit message: Reworked the board to work with the BC805M module
Parts:
- C3: footprint Capacitor_SMD:C_0805_2012Metric_Pad1.15x1.40mm_HandSolder -> Capacitor_SMD:C_0805_2012Metric_Pad1.18x1.45mm_HandSolder
Changed lines of the file:
@@
 F 0 "C3" H 6665 1296 50  0000 L CNN
 F 1 "2.2uF" H 6665 1205 50  0000 L CNN
-F 2 "Capacitor_SMD:C_0805_2012Metric_Pad1.15x1.40mm_HandSolder" H 6588 1100 50  0001 C CNN
+F 2 "Capacitor_SMD:C_0805_2012Metric_Pad1.18x1.45mm_HandSolder" H 6588 1100 50  0001 C CNN
 F 3 "~" H 6550 1250 50  0001 C CNN
 	1    6550 1250
@@
 	6550 1050 6900 1050
 $Comp
-L power:+2V8 #PWR?
+L power:+2V8 #PWR0101
 U 1 1 61153FAD
 P 2050 950
-F 0 "#PWR?" H 2050 800 50  0001 C CNN
+F 0 "#PWR0101" H 2050 800 50  0001 C CNN
 F 1 "+2V8" H 2065 1123 50  0000 C CNN
 F 2 "" H 2050 950 50  0001 C CNN
@@
 $EndComp
 $Comp
-L power:+2V8 #PWR?
+L power:+2V8 #PWR0104
 U 1 1 611582E1
 P 3100 950
-F 0 "#PWR?" H 3100 800 50  0001 C CNN
+F 0 "#PWR0104" H 3100 800 50  0001 C CNN
 F 1 "+2V8" H 3115 1123 50  0000 C CNN
 F 2 "" H 3100 950 50  0001 C CNN
@@
 $EndComp
 $Comp
-L power:+2V8 #PWR?
+L power:+2V8 #PWR0115
 U 1 1 6115E2AE
 P 5050 2400
-F 0 "#PWR?" H 5050 2250 50  0001 C CNN
+F 0 "#PWR0115" H 5050 2250 50  0001 C CNN
 F 1 "+2V8" H 5065 2573 50  0000 C CNN
 F 2 "" H 5050 2400 50  0001 C CNN
@@
 $EndComp
 $Comp
-L power:+2V8 #PWR?
+L power:+2V8 #PWR0118
 U 1 1 61161DBD
 P 7150 2050
-F 0 "#PWR?" H 7150 1900 50  0001 C CNN
+F 0 "#PWR0118" H 7150 1900 50  0001 C CNN
 F 1 "+2V8" H 7165 2223 50  0000 C CNN
 F 2 "" H 7150 2050 50  0001 C CNN
@@
 	7625 2050 7150 2050
 $Comp
-L power:+2V8 #PWR?
+L power:+2V8 #PWR0121
 U 1 1 6119B4C5
 P 6850 3800
-F 0 "#PWR?" H 6850 3650 50  0001 C CNN
+F 0 "#PWR0121" H 6850 3650 50  0001 C CNN
 F 1 "+2V8" H 6865 3973 50  0000 C CNN
 F 2 "" H 6850 3800 50  0001 C CNN
